File: hardware/frontend_wifi.kicad_sch (KiCad schematic)
At the start: 9 parts

Commit message: jamrf-v2: Add U3V70F15 WiFi PA regulator, FR408HR stackup, full firmware, custom footprints
- Add U3V70F15 buck-boost converter to limit WiFi PA supply to 15V (fixes ZVE-3W-83+ overvoltage)
- Update PCB stackup to Isola FR408HR (Er=3.65, tan d=0.0095) with corrected 0.40mm 50-ohm traces
- Add full operational firmware (main.py): chaos modulation engine, ST7789 display, mode control
- Add 6 custom footprints: M5StickC, Pololu D24V10F5/U3V70F15, Mini-Circuits, Wurth shield, isolator
- Add fp-lib-table and sym-lib-table for custom libraries
- Update README with logo, badges, TIIUAE disclaimer, corrected specs
- Update LICENSE with proper attribution

Co-Authored-By: Claude Opus 4.6 <noreply@anthropic.com>
Parts:
- C?: renamed from C_VCO?; value 100nF -> C
- ISO?: value B2425 -> Ferrite_Isolator
- J?: value SMA WiFi -> SMA
- R? (x2): value 292R -> R
- R?: value 18R -> R
Changed lines of the file:
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@@
 	(text "WiFi 2.4 GHz RF Chain\nSignal flow: VCO -> Pi-Atten (3dB) -> BPF -> WiFi PA (3W) -> Isolator -> SMA\n50-ohm controlled impedance throughout"
 		(exclude_from_sim no)
-		(at 40.64 40.64 0)
+		(at 37.338 33.274 0)
 		(effects
 			(font
@@
 		(on_board yes)
 		(dnp no)
-		(property "Reference" "C_VCO?"
+		(property "Reference" "C?"
 			(at 50.8 60.96 90)
 			(effects
@@
 			)
 		)
-		(property "Value" "100nF"
+		(property "Value" "C"
 			(at 45.72 60.96 90)
 			(effects
@@
 			)
 		)
-		(property "Description" ""
+		(property "Description" "Unpolarized capacitor"
 			(at 48.26 60.96 0)
 			(effects
@@
 			(project "jamrf-v2"
 				(path "/b0000001-0000-0000-0000-000000000001/b0000001-0000-0000-0000-000000000030"
-					(reference "C_VCO?")
+					(reference "C?")
 					(unit 1)
 				)
@@
 			)
 		)
-		(property "Value" "292R"
+		(property "Value" "R"
 			(at 81.28 76.2 90)
 			(effects
@@
 			)
 		)
-		(property "Description" ""
+		(property "Description" "Resistor"
 			(at 83.82 76.2 0)
 			(effects
@@
 			)
 		)
-		(property "Value" "18R"
+		(property "Value" "R"
 			(at 96.52 74.93 0)
 			(effects
@@
 			)
 		)
-		(property "Description" ""
+		(property "Description" "Resistor"
 			(at 96.52 72.39 0)
 			(effects
@@
 			)
 		)
-		(property "Value" "292R"
+		(property "Value" "R"
 			(at 106.68 76.2 90)
 			(effects
@@
 			)
 		)
-		(property "Description" ""
+		(property "Description" "Resistor"
 			(at 109.22 76.2 0)
 			(effects
@@
 			)
 		)
-		(property "Value" "B2425"
+		(property "Value" "Ferrite_Isolator"
 			(at 203.2 82.55 0)
 			(effects
@@
 			)
 		)
-		(property "Value" "SMA WiFi"
+		(property "Value" "SMA"
 			(at 231.14 81.28 0)
 			(effects

Commit message: Annotate all component references and update CLAUDE.md
- All component references annotated (U1-U10, R1-R17, C1-C19, Q1-Q4, etc.)
- Fix CLAUDE.md: correct jamrf-v4 description (dual-band, not WiFi-only)
- Update CLAUDE.md: file paths match main branch structure, add firmware docs
- Remove resolved known issues (annotation, footprint library)

Co-Authored-By: Claude Opus 4.6 <noreply@anthropic.com>
Parts:
- gave numbers to parts that had none: 9
Changed lines of the file:
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@@
 		(on_board yes)
 		(dnp no)
-		(property "Reference" "U?"
+		(property "Reference" "U4"
 			(at 55.88 64.77 0)
 			(effects
@@
 			(project "jamrf-v2"
 				(path "/b0000001-0000-0000-0000-000000000001/b0000001-0000-0000-0000-000000000030"
-					(reference "U?")
+					(reference "U4")
 					(unit 1)
 				)
@@
 		(on_board yes)
 		(dnp no)
-		(property "Reference" "C?"
+		(property "Reference" "C4"
 			(at 50.8 60.96 90)
 			(effects
@@
 			(project "jamrf-v2"
 				(path "/b0000001-0000-0000-0000-000000000001/b0000001-0000-0000-0000-000000000030"
-					(reference "C?")
+					(reference "C4")
 					(unit 1)
 				)
@@
 		(on_board yes)
 		(dnp no)
-		(property "Reference" "R?"
+		(property "Reference" "R6"
 			(at 86.36 76.2 90)
 			(effects
@@
 			(project "jamrf-v2"
 				(path "/b0000001-0000-0000-0000-000000000001/b0000001-0000-0000-0000-000000000030"
-					(reference "R?")
+					(reference "R6")
 					(unit 1)
 				)
@@
 		(on_board yes)
 		(dnp no)
-		(property "Reference" "R?"
+		(property "Reference" "R7"
 			(at 96.52 69.85 0)
 			(effects
@@
 			(project "jamrf-v2"
 				(path "/b0000001-0000-0000-0000-000000000001/b0000001-0000-0000-0000-000000000030"
-					(reference "R?")
+					(reference "R7")
 					(unit 1)
 				)
@@
 		(on_board yes)
 		(dnp no)
-		(property "Reference" "R?"
+		(property "Reference" "R8"
 			(at 111.76 76.2 90)
 			(effects
@@
 			(project "jamrf-v2"
 				(path "/b0000001-0000-0000-0000-000000000001/b0000001-0000-0000-0000-000000000030"
-					(reference "R?")
+					(reference "R8")
 					(unit 1)
 				)
@@
 		(on_board yes)
 		(dnp no)
-		(property "Reference" "F?"
+		(property "Reference" "F2"
 			(at 132.08 69.85 0)
 			(effects
@@
 			(project "jamrf-v2"
 				(path "/b0000001-0000-0000-0000-000000000001/b0000001-0000-0000-0000-000000000030"
-					(reference "F?")
+					(reference "F2")
 					(unit 1)
 				)
@@
 		(on_board yes)
 		(dnp no)
-		(property "Reference" "U?"
+		(property "Reference" "U5"
 			(at 167.64 64.77 0)
 			(effects
@@
 			(project "jamrf-v2"
 				(path "/b0000001-0000-0000-0000-000000000001/b0000001-0000-0000-0000-000000000030"
-					(reference "U?")
+					(reference "U5")
 					(unit 1)
 				)
@@
 		(on_board yes)
 		(dnp no)
-		(property "Reference" "ISO?"
+		(property "Reference" "ISO2"
 			(at 203.2 69.85 0)
 			(effects
@@
 			(project "jamrf-v2"
 				(path "/b0000001-0000-0000-0000-000000000001/b0000001-0000-0000-0000-000000000030"
-					(reference "ISO?")
+					(reference "ISO2")
 					(unit 1)
 				)
@@
 		(on_board yes)
 		(dnp no)
-		(property "Reference" "J?"
+		(property "Reference" "J2"
 			(at 231.14 71.12 0)
 			(effects
@@
 			(project "jamrf-v2"
 				(path "/b0000001-0000-0000-0000-000000000001/b0000001-0000-0000-0000-000000000030"
-					(reference "J?")
-					(unit 1)
-				)
+					(reference "J2")
+					(unit 1)
+				)
